Commit message: modifications for self collision

File: data/urdf/rh56dfx_left.urdf (robot description, URDF)
Before this commit: robot rh56dfx, 37 links, 36 joints
Links:
- link left_index_rubber_1: geometry visual mesh filename=/workspace/external/rh56dfx_description/meshes/left/visual/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
- link left_index_rubber_2: geometry visual mesh filename=/workspace/external/rh56dfx_description/meshes/left/visual/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
- link left_little_rubber_1: geometry visual mesh filename=/workspace/external/rh56dfx_description/meshes/left/visual/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
- link left_little_rubber_2: geometry visual mesh filename=/workspace/external/rh56dfx_description/meshes/left/visual/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
- link left_middle_rubber_1: geometry visual mesh filename=/workspace/external/rh56dfx_description/meshes/left/visual/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
- link left_middle_rubber_2: geometry visual mesh filename=/workspace/external/rh56dfx_description/meshes/left/visual/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
- link left_ring_rubber_1: geometry visual mesh filename=/workspace/external/rh56dfx_description/meshes/left/visual/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
- link left_ring_rubber_2: geometry visual mesh filename=/workspace/external/rh56dfx_description/meshes/left/visual/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
- link left_thumb_rubber_1: geometry visual mesh filename=/workspace/external/rh56dfx_description/meshes/left/visual/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
- link left_thumb_rubber_2: geometry visual mesh filename=/workspace/external/rh56dfx_description/meshes/left/visual/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
- link left_thumb_rubber_3: geometry visual mesh filename=/workspace/external/rh56dfx_description/meshes/left/visual/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

File: data/urdf/rh56dfx_right.urdf (robot description, URDF)
Before this commit: robot rh56dfx, 37 links, 36 joints
Links:
- link right_index_rubber_1: geometry visual mesh filename=/workspace/external/rh56dfx_description/meshes/right/visual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
- link right_index_rubber_2: geometry visual mesh filename=/workspace/external/rh56dfx_description/meshes/right/visual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
- link right_little_rubber_1: geometry visual mesh filename=/workspace/external/rh56dfx_description/meshes/right/visual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
- link right_little_rubber_2: geometry visual mesh filename=/workspace/external/rh56dfx_description/meshes/right/visual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
- link right_middle_rubber_1: geometry visual mesh filename=/workspace/external/rh56dfx_description/meshes/right/visual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
- link right_middle_rubber_2: geometry visual mesh filename=/workspace/external/rh56dfx_description/meshes/right/visual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
- link right_ring_rubber_1: geometry visual mesh filename=/workspace/external/rh56dfx_description/meshes/right/visual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
- link right_ring_rubber_2: geometry visual mesh filename=/workspace/external/rh56dfx_description/meshes/right/visual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
- link right_thumb_rubber_1: geometry visual mesh filename=/workspace/external/rh56dfx_description/meshes/right/visual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
- link right_thumb_rubber_2: geometry visual mesh filename=/workspace/external/rh56dfx_description/meshes/right/visual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
- link right_thumb_rubber_3: geometry visual mesh filename=/workspace/external/rh56dfx_description/meshes/right/visual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

Commit message: collision fixes

File: data/urdf/rh56dfx_left.urdf (robot description, URDF)
Before this commit: robot rh56dfx, 37 links, 36 joints
Links:
- link left_index_rubber_1: geometry collision mesh filename=/workspace/external/rh56dfx_description/meshes/left/collisi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; visual mesh filename=/workspace/external/rh56dfx_description/meshes/left/visual/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
- link left_index_rubber_2: geometry collision mesh filename=/workspace/external/rh56dfx_description/meshes/left/collisi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; visual mesh filename=/workspace/external/rh56dfx_description/meshes/left/visual/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
- link left_little_rubber_1: geometry collision mesh filename=/workspace/external/rh56dfx_description/meshes/left/collisi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; visual mesh filename=/workspace/external/rh56dfx_description/meshes/left/visual/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
- link left_little_rubber_2: geometry collision mesh filename=/workspace/external/rh56dfx_description/meshes/left/collisi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; visual mesh filename=/workspace/external/rh56dfx_description/meshes/left/visual/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
- link left_middle_rubber_1: geometry collision mesh filename=/workspace/external/rh56dfx_description/meshes/left/collisi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; visual mesh filename=/workspace/external/rh56dfx_description/meshes/left/visual/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
- link left_middle_rubber_2: geometry collision mesh filename=/workspace/external/rh56dfx_description/meshes/left/collisi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; visual mesh filename=/workspace/external/rh56dfx_description/meshes/left/visual/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
- link left_ring_rubber_1: geometry collision mesh filename=/workspace/external/rh56dfx_description/meshes/left/collisi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; visual mesh filename=/workspace/external/rh56dfx_description/meshes/left/visual/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
- link left_ring_rubber_2: geometry collision mesh filename=/workspace/external/rh56dfx_description/meshes/left/collisi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; visual mesh filename=/workspace/external/rh56dfx_description/meshes/left/visual/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
- link left_thumb_rubber_1: geometry collision mesh filename=/workspace/external/rh56dfx_description/meshes/left/collisi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; visual mesh filename=/workspace/external/rh56dfx_description/meshes/left/visual/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
- link left_thumb_rubber_2: geometry collision mesh filename=/workspace/external/rh56dfx_description/meshes/left/collisi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; visual mesh filename=/workspace/external/rh56dfx_description/meshes/left/visual/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
- link left_thumb_rubber_3: geometry collision mesh filename=/workspace/external/rh56dfx_description/meshes/left/collisi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; visual mesh filename=/workspace/external/rh56dfx_description/meshes/left/visual/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

File: data/urdf/rh56dfx_right.urdf (robot description, URDF)
Before this commit: robot rh56dfx, 37 links, 36 joints
Links:
- link right_index_rubber_1: geometry collision mesh filename=/workspace/external/rh56dfx_description/meshes/right/collis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; visual mesh filename=/workspace/external/rh56dfx_description/meshes/right/visual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
- link right_index_rubber_2: geometry collision mesh filename=/workspace/external/rh56dfx_description/meshes/right/collis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; visual mesh filename=/workspace/external/rh56dfx_description/meshes/right/visual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
- link right_little_rubber_1: geometry collision mesh filename=/workspace/external/rh56dfx_description/meshes/right/collis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; visual mesh filename=/workspace/external/rh56dfx_description/meshes/right/visual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
- link right_little_rubber_2: geometry collision mesh filename=/workspace/external/rh56dfx_description/meshes/right/collis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; visual mesh filename=/workspace/external/rh56dfx_description/meshes/right/visual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
- link right_middle_rubber_1: geometry collision mesh filename=/workspace/external/rh56dfx_description/meshes/right/collis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; visual mesh filename=/workspace/external/rh56dfx_description/meshes/right/visual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
- link right_middle_rubber_2: geometry collision mesh filename=/workspace/external/rh56dfx_description/meshes/right/collis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; visual mesh filename=/workspace/external/rh56dfx_description/meshes/right/visual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
- link right_ring_rubber_1: geometry collision mesh filename=/workspace/external/rh56dfx_description/meshes/right/collis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; visual mesh filename=/workspace/external/rh56dfx_description/meshes/right/visual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
- link right_ring_rubber_2: geometry collision mesh filename=/workspace/external/rh56dfx_description/meshes/right/collis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; visual mesh filename=/workspace/external/rh56dfx_description/meshes/right/visual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
- link right_thumb_rubber_1: geometry collision mesh filename=/workspace/external/rh56dfx_description/meshes/right/collis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; visual mesh filename=/workspace/external/rh56dfx_description/meshes/right/visual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
- link right_thumb_rubber_2: geometry collision mesh filename=/workspace/external/rh56dfx_description/meshes/right/collis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; visual mesh filename=/workspace/external/rh56dfx_description/meshes/right/visual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
- link right_thumb_rubber_3: geometry collision mesh filename=/workspace/external/rh56dfx_description/meshes/right/collis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; visual mesh filename=/workspace/external/rh56dfx_description/meshes/right/visual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
